File: exocam_charge_amp.sch (KiCad schematic (older format))
At the start: 17 parts, among them J1 jstsh6x1, U1 TLV2771CDBVT, U2 TLV2771CDBVT

Commit message: updated pcb to mostly reflect double amp
Parts:
- BZ2: footprint exocam_charge_amp:piezo_buzzer -> exocam_charge_amp:piezo_buzzer_alt
- J1: footprint (none) -> exocam_charge_amp:jstsh6x1
Changed lines of the file:
@@
 F 0 "BZ2" V 1951 3363 50  0000 R CNN
 F 1 "Buzzer" V 1860 3363 50  0000 R CNN
-F 2 "exocam_charge_amp:piezo_buzzer" V 1875 3650 50  0001 C CNN
+F 2 "exocam_charge_amp:piezo_buzzer_alt" V 1875 3650 50  0001 C CNN
 F 3 "~" V 1875 3650 50  0001 C CNN
 	1    1900 3550
@@
 $EndComp
 $Comp
-L power:GND #PWR?
+L power:GND #PWR0101
 U 1 1 60DFD440
 P 2950 4350
-F 0 "#PWR?" H 2950 4100 50  0001 C CNN
+F 0 "#PWR0101" H 2950 4100 50  0001 C CNN
 F 1 "GND" V 2955 4222 50  0000 R CNN
 F 2 "" H 2950 4350 50  0001 C CNN
@@
 F 0 "J1" V 4304 522 50  0000 R CNN
 F 1 "jstsh6x1" V 4213 522 50  0000 R CNN
-F 2 "" H 4200 1300 50  0001 C CNN
+F 2 "exocam_charge_amp:jstsh6x1" H 4200 1300 50  0001 C CNN
 F 3 "" H 4200 1300 50  0001 C CNN
 	1    4250 1150
@@
 $EndComp
 $Comp
-L power:+3.3V #PWR?
+L power:+3.3V #PWR0104
 U 1 1 60E1C732
 P 4800 1000
-F 0 "#PWR?" H 4800 850 50  0001 C CNN
+F 0 "#PWR0104" H 4800 850 50  0001 C CNN
 F 1 "+3.3V" H 4815 1173 50  0000 C CNN
 F 2 "" H 4800 1000 50  0001 C CNN
@@
 	4800 1050 4800 1000
 $Comp
-L power:GND #PWR?
+L power:GND #PWR0105
 U 1 1 60E1EDAD
 P 4150 950
-F 0 "#PWR?" H 4150 700 50  0001 C CNN
+F 0 "#PWR0105" H 4150 700 50  0001 C CNN
 F 1 "GND" H 4155 777 50  0000 C CNN
 F 2 "" H 4150 950 50  0001 C CNN
@@
 AMP2
 $Comp
-L power:+3.3V #PWR?
+L power:+3.3V #PWR0106
 U 1 1 60E36A79
 P 3800 4250
-F 0 "#PWR?" H 3800 4100 50  0001 C CNN
+F 0 "#PWR0106" H 3800 4100 50  0001 C CNN
 F 1 "+3.3V" H 3815 4423 50  0000 C CNN
 F 2 "" H 3800 4250 50  0001 C CNN
@@
 	3700 4250 3800 4250
 $Comp
-L power:+3.3V #PWR?
+L power:+3.3V #PWR0107
 U 1 1 60E3956C
 P 3750 1500
-F 0 "#PWR?" H 3750 1350 50  0001 C CNN
+F 0 "#PWR0107" H 3750 1350 50  0001 C CNN
 F 1 "+3.3V" H 3765 1673 50  0000 C CNN
 F 2 "" H 3750 1500 50  0001 C CNN
@@
 	1700 1200 1700 1950
 $Comp
-L power:+3.3V #PWR?
+L power:+3.3V #PWR0108
 U 1 1 60E3E4A9
 P 900 1000
-F 0 "#PWR?" H 900 850 50  0001 C CNN
+F 0 "#PWR0108" H 900 850 50  0001 C CNN
 F 1 "+3.3V" H 915 1173 50  0000 C CNN
 F 2 "" H 900 1000 50  0001 C CNN
