File: exocam_charge_amp.kicad_pcb (KiCad board)
At the start: 2 copper layers, 29.6 x 18 mm, 12 parts, among them J1 dupont4x1, U1 TLV2771CDBVT

Commit message: updated pcb to mostly reflect double amp
Parts:
- added BZ2: Buzzer, exocam_charge_amp:piezo_buzzer_alt, F.Cu at (76.5, 64.3)
- added C2: 5pF, exocam_charge_amp:0603_R, F.Cu at (69.8, 64.0)
- added R5: 1M, exocam_charge_amp:0603_R, F.Cu at (69.3, 63.0)
- added R6: 1M, exocam_charge_amp:0603_R, F.Cu at (69.1, 65.6)
- added U2: TLV2771CDBVT, exocam_charge_amp:TLV2271DBV, F.Cu at (70.5, 63.2)
- J1: value dupont4x1 -> jstsh6x1; footprint exocam_charge_amp:dupont4x1 -> exocam_charge_amp:jstsh6x1
- moved R2 21.9 mm to (46.2, 62.2), turned to 90 degrees
- moved R1 15.3 mm to (46.2, 65.3), turned to 90 degrees
- moved J1 6.55 mm to (61.2, 66.2), turned to 0 degrees
- moved R4 4.89 mm to (61.1, 59.8), turned to 90 degrees
- moved BZ1 4.78 mm to (58.0, 60.7), turned to 270 degrees
- moved U1 3.88 mm to (58.7, 62.9), turned to 270 degrees
- moved R3 2.70 mm to (56.6, 62.5), turned to 180 degrees
- moved C1 2.42 mm to (56.6, 61.1), turned to 180 degrees
Connections:
- net /Amplified renamed AMP1
- net /UnAmplified renamed UNAMP1
- net Net-(BZ1-Pad2) renamed VGND
- J1 pad 4: +5V -> AMP2
- R1 pad 1: +5V -> +3V3
- U1 pad 5: +5V -> +3V3
Routing:
- net +3V3: track 0.00 -> 26.9 mm
- net AMP2: track 0.00 -> 18.5 mm
- net VGND: track 20.2 -> 38.0 mm, vias 2 -> 4
- net UNAMP2: track 0.00 -> 17.0 mm
- net GND: track 11.8 -> 28.6 mm
- net +5V: track 9.25 -> 0.00 mm
- net UNAMP1: track 19.7 -> 25.2 mm, vias 2 -> 5
- net AMP1: track 15.4 -> 11.6 mm, vias 2 -> 0

Commit message: updated shoulder to include the 3 amps
Parts:
- added BZ3: Buzzer, exocam_charge_amp:jstsh2x1, F.Cu at (53.7, 66.6)
- added C3: 5pF, exocam_charge_amp:0603_R, F.Cu at (55.4, 59.5)
- added R7: 1M, exocam_charge_amp:0603_R, B.Cu at (50.9, 63.8)
- added R8: 1M, exocam_charge_amp:0603_R, F.Cu at (55.4, 58.0)
- added U3: TLV2771CDBVT, exocam_charge_amp:TLV2271DBV, F.Cu at (55.1, 67.9)
- BZ1: footprint exocam_charge_amp:piezo_buzzer -> exocam_charge_amp:piezo_buzzer_alt
- BZ2: footprint exocam_charge_amp:piezo_buzzer_alt -> exocam_charge_amp:jstsh2x1
- C1, R1, R2, R3, R4, R5, U1: moved to B.Cu
- J1: value jstsh6x1 -> jstsh8x1; footprint exocam_charge_amp:jstsh6x1 -> exocam_charge_amp:jstsh8x1
- moved R1 15.7 mm to (61.5, 68.7), turned to 180 degrees
- moved R2 13.8 mm to (58.4, 68.7), turned to 180 degrees
- moved BZ2 9.12 mm to (67.7, 62.0), turned to 90 degrees
- moved U1 7.68 mm to (62.1, 56.0), turned to 180 degrees
- moved R3 7.14 mm to (62.6, 66.3), turned to 0 degrees
- moved C1 6.96 mm to (62.6, 64.7), turned to 0 degrees
- moved C2 6.66 mm to (66.3, 69.6)
- moved R6 6.09 mm to (66.3, 71.0)
- moved U2 4.74 mm to (66.2, 61.1), turned to 0 degrees
- moved R4 3.56 mm to (57.6, 59.0)
- moved BZ1 3.13 mm to (55.0, 59.9)
- moved R5 2.13 mm to (70.2, 65.0), turned to 270 degrees
- moved J1 1.46 mm to (59.7, 66.2)
Connections:
- J1 pad 6: +3V3 -> AMP3
- J1 pad 7: (no net) -> UNAMP3
Routing:
- net UNAMP3: track 0.00 -> 28.2 mm, vias 0 -> 1
- net VGND: track 38.0 -> 59.7 mm, vias 4 -> 5
- net AMP3: track 0.00 -> 21.5 mm, vias 0 -> 2
- net +3V3: track 26.9 -> 46.1 mm, vias 0 -> 4
- net UNAMP1: track 25.2 -> 17.3 mm, vias 5 -> 1
- net GND: track 28.6 -> 33.4 mm, vias 2 -> 3
- net AMP1: track 11.6 -> 16.4 mm, vias 0 -> 5
- net AMP2: track 18.5 -> 15.3 mm
- net UNAMP2: track 17.0 -> 19.8 mm, vias 0 -> 1
