File: main_board/main_board/main_board.kicad_pcb (KiCad board)
At the start: 2 copper layers, 78.1 x 27.4 mm, 26 parts, among them J1 jstsh4x1, J2 3.3v bus, J3 GND_bus, U1 Teensy3.5_All_Pins, U2 TLV2771CDBVT, U3 TLV2771CDBVT, U4 TLV2771CDBVT

Commit message: updated pinout for daughter board (changed pin for AMP3)
Connections:
- U1 pad 43: AMP3 -> Net-(U1-Pad43)
- U1 pad 57: Net-(U1-Pad57) -> AMP3
